File: EAGLE/projects/CAN-D Rev2/CAN-D Coat Rev1.sch (EAGLE design)
At the start: 14 parts, among them J1 TSM-106-SV, J2 TSM-106-SV

Commit message: Clean up EAGLE files
Parts:
- DS1, DS2, DS3, PWRLED: value L130-6580001400001 -> LED; device L130-6580001400001:L130-6580001400001 -> CAN-D:LED
- J1, J2: value TSM-106-SV -> RECEPTACLE; device con-samtec:TSM-106-SV -> CAN-D:RECEPTACLE
- JTAG: value SAMTEC-TSM-110-01-X-DVJ -> JTAG-HEADERJ; device SAMTEC-TSM-110-01-X-DV:SAMTEC-TSM-110-01-X-DVJ -> CAN-D:JTAG-HEADERJ
- LOG, MARK: value SCHURTER-LSH-1301.9314 -> BUTTONSPLUNGER; device schurter_switches_LSH_SMS:SCHURTER-LSH-1301.9314 -> CAN-D:BUTTONSPLUNGER
- R1, R2, R4: device rcl:R-US_R0603 -> CAN-D:RESISTOR
- RESET: value SCHURTER-LSH-1301.9314 -> BUTTONS; device schurter_switches_LSH_SMS:SCHURTER-LSH-1301.9314 -> CAN-D:BUTTONS
Changed lines of the file:
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@@
 <?xml version="1.0" encoding="utf-8"?>
 <!DOCTYPE eagle SYSTEM "eagle.dtd">
-<eagle version="9.3.1">
+<eagle version="9.3.2">
 <drawing>
 <settings>
@@
 </classes>
 <parts>
-<part name="JTAG" library="SAMTEC-TSM-110-01-X-DV" deviceset="SAMTEC-TSM-110-01-X-DV" device="J"/>
-<part name="LOG" library="schurter_switches_LSH_SMS" deviceset="SCHURTER-LSH-*" device="" technology="1301.9314"/>
-<part name="MARK" library="schurter_switches_LSH_SMS" deviceset="SCHURTER-LSH-*" device="" technology="1301.9314"/>
-<part name="RESET" library="schurter_switches_LSH_SMS" deviceset="SCHURTER-LSH-*" device="" technology="1301.9314"/>
-<part name="DS1" library="L130-6580001400001" deviceset="L130-6580001400001" device=""/>
-<part name="DS2" library="L130-6580001400001" deviceset="L130-6580001400001" device=""/>
-<part name="DS3" library="L130-6580001400001" deviceset="L130-6580001400001" device=""/>
-<part name="PWRLED" library="L130-6580001400001" deviceset="L130-6580001400001" device=""/>
-<part name="J1" library="con-samtec" deviceset="TSM-106-SV" device=""/>
-<part name="J2" library="con-samtec" deviceset="TSM-106-SV" device=""/>
+<part name="JTAG" library="CAN-D" library_urn="urn:adsk.eagle:library:10031387" deviceset="JTAG-HEADER" device="J" package3d_urn="urn:adsk.eagle:package:10031773/5"/>
+<part name="LOG" library="CAN-D" library_urn="urn:adsk.eagle:library:10031387" deviceset="BUTTONS" device="PLUNGER" package3d_urn="urn:adsk.eagle:package:10045811/3" value="BUTTONSPLUNGER"/>
+<part name="MARK" library="CAN-D" library_urn="urn:adsk.eagle:library:10031387" deviceset="BUTTONS" device="PLUNGER" package3d_urn="urn:adsk.eagle:package:10045811/3" value="BUTTONSPLUNGER"/>
+<part name="RESET" library="CAN-D" library_urn="urn:adsk.eagle:library:10031387" deviceset="BUTTONS" device="" package3d_urn="urn:adsk.eagle:package:10031812/2"/>
+<part name="DS1" library="CAN-D" library_urn="urn:adsk.eagle:library:10031387" deviceset="LED" device="" package3d_urn="urn:adsk.eagle:package:10031816/2"/>
+<part name="DS2" library="CAN-D" library_urn="urn:adsk.eagle:library:10031387" deviceset="LED" device="" package3d_urn="urn:adsk.eagle:package:10031816/2"/>
+<part name="DS3" library="CAN-D" library_urn="urn:adsk.eagle:library:10031387" deviceset="LED" device="" package3d_urn="urn:adsk.eagle:package:10031816/2"/>
+<part name="PWRLED" library="CAN-D" library_urn="urn:adsk.eagle:library:10031387" deviceset="LED" device="" package3d_urn="urn:adsk.eagle:package:10031816/2"/>
+<part name="J1" library="CAN-D" library_urn="urn:adsk.eagle:library:10031387" deviceset="RECEPTACLE" device="" package3d_urn="urn:adsk.eagle:package:10031897/2"/>
+<part name="J2" library="CAN-D" library_urn="urn:adsk.eagle:library:10031387" deviceset="RECEPTACLE" device="" package3d_urn="urn:adsk.eagle:package:10031897/2"/>
 <part name="GND1" library="supply1" library_urn="urn:adsk.eagle:library:371" deviceset="GND" device=""/>
 <part name="GND2" library="supply1" library_urn="urn:adsk.eagle:library:371" deviceset="GND" device=""/>
 <part name="GND3" library="supply1" library_urn="urn:adsk.eagle:library:371" deviceset="GND" device=""/>
 <part name="GND4" library="supply1" library_urn="urn:adsk.eagle:library:371" deviceset="GND" device=""/>
-<part name="R1" library="rcl" library_urn="urn:adsk.eagle:library:334" deviceset="R-US_" device="R0603" package3d_urn="urn:adsk.eagle:package:23555/3" value="550"/>
-<part name="R2" library="rcl" library_urn="urn:adsk.eagle:library:334" deviceset="R-US_" device="R0603" package3d_urn="urn:adsk.eagle:package:23555/3" value="550"/>
+<part name="R1" library="CAN-D" library_urn="urn:adsk.eagle:library:10031387" deviceset="RESISTOR" device="" package3d_urn="urn:adsk.eagle:package:23555/3" value="550"/>
+<part name="R2" library="CAN-D" library_urn="urn:adsk.eagle:library:10031387" deviceset="RESISTOR" device="" package3d_urn="urn:adsk.eagle:package:23555/3" value="550"/>
 <part name="R3" library="rcl" library_urn="urn:adsk.eagle:library:334" deviceset="R-US_" device="R0603" package3d_urn="urn:adsk.eagle:package:23555/3" value="550"/>
-<part name="R4" library="rcl" library_urn="urn:adsk.eagle:library:334" deviceset="R-US_" device="R0603" package3d_urn="urn:adsk.eagle:package:23555/3" value="550"/>
+<part name="R4" library="CAN-D" library_urn="urn:adsk.eagle:library:10031387" deviceset="RESISTOR" device="" package3d_urn="urn:adsk.eagle:package:23555/3" value="550"/>
 <part name="P+1" library="supply1" library_urn="urn:adsk.eagle:library:371" deviceset="VCC" device=""/>
 </parts>
