File: EAGLE/projects/CAN-D Rev2/CAN-D Coat Rev2.brd (EAGLE design)
At the start: 55.3 x 80.3 mm, 14 parts, among them J1 RECEPTACLE, J2 RECEPTACLE

Commit message: Upload Final Revisions to Board Design
Parts:
- JTAG: device CAN-D:TSM-110-02-L-DV-A-P-TR -> CAN-D:TSM-110-02-S-DV-P-TR
Connections:
- net LED1: now also J2.4; no longer J2.3
- net LED2: now also J2.5; no longer J2.2
- net LED3: now also J2.6; no longer J2.1
- net LOG: now also J2.3; no longer J2.4
- net MARK: now also J2.2; no longer J2.5
- net RESET: now also J2.1; no longer J2.6
Routing:
- net LED3: track 33.7 -> 56.3 mm
- net RESET: track 44.9 -> 34.7 mm
- net LED1: track 31.2 -> 39.2 mm
- net LOG: track 90.7 -> 97.7 mm
- net MARK: track 38.8 -> 45.6 mm
- net LED2: track 35.2 -> 37.4 mm
Other:
- board text added: "CAN-D Coating Rev2"
- board text added: "LED1"
- board text added: "LED2"
- board text added: "LED3"
- board text added: "LOG"
- board text added: "MARK"
- board text added: "RESET"
- board text removed: "CAN-D Coating Rev1"
