File: EAGLE/projects/CAN-D Rev2/CAN-D Coat Rev2.sch (EAGLE design)
At the start: 14 parts, among them J1 RECEPTACLE, J2 RECEPTACLE

Commit message: Upload Final Revisions to Board Design
Connections:
- net LED1: now also J2.4; no longer J2.3
- net LED2: now also J2.5; no longer J2.2
- net LED3: now also J2.6; no longer J2.1
- net LOG: now also J2.3; no longer J2.4
- net MARK: now also J2.2; no longer J2.5
- net RESET: now also J2.1; no longer J2.6
Other:
- note added: "CAN-D Coating Rev2"
Changed lines of the file:
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@@
 </classes>
 <parts>
-<part name="JTAG" library="CAN-D" library_urn="urn:adsk.eagle:library:10031387" deviceset="JTAG-HEADER" device="J" package3d_urn="urn:adsk.eagle:package:10031773/5"/>
+<part name="JTAG" library="CAN-D" library_urn="urn:adsk.eagle:library:10031387" deviceset="JTAG-HEADER" device="J" package3d_urn="urn:adsk.eagle:package:10031773/6"/>
 <part name="LOG" library="CAN-D" library_urn="urn:adsk.eagle:library:10031387" deviceset="BUTTONS" device="PLUNGER" package3d_urn="urn:adsk.eagle:package:10045811/3" value="BUTTONSPLUNGER"/>
 <part name="MARK" library="CAN-D" library_urn="urn:adsk.eagle:library:10031387" deviceset="BUTTONS" device="PLUNGER" package3d_urn="urn:adsk.eagle:package:10045811/3" value="BUTTONSPLUNGER"/>
@@
 <sheet>
 <plain>
+<text x="58.42" y="38.1" size="1.778" layer="91">CAN-D Coating Rev2</text>
 </plain>
 <instances>
@@
 <net name="LED3" class="0">
 <segment>
-<pinref part="J2" gate="G$1" pin="1"/>
-<wire x1="129.54" y1="83.82" x2="127" y2="83.82" width="0.1524" layer="91"/>
-<label x="121.92" y="83.82" size="1.778" layer="95"/>
-</segment>
-<segment>
 <pinref part="R3" gate="G$1" pin="1"/>
 <wire x1="111.76" y1="7.62" x2="106.68" y2="7.62" width="0.1524" layer="91"/>
 <label x="101.6" y="7.62" size="1.778" layer="95"/>
 </segment>
+<segment>
+<pinref part="J2" gate="G$1" pin="6"/>
+<wire x1="129.54" y1="71.12" x2="127" y2="71.12" width="0.1524" layer="91"/>
+<label x="121.92" y="71.12" size="1.778" layer="95"/>
+</segment>
 </net>
 <net name="LED2" class="0">
-<segment>
-<pinref part="J2" gate="G$1" pin="2"/>
-<wire x1="129.54" y1="81.28" x2="127" y2="81.28" width="0.1524" layer="91"/>
-<label x="121.92" y="81.28" size="1.778" layer="95"/>
-</segment>
 <segment>
 <pinref part="R2" gate="G$1" pin="1"/>
@@
 <label x="101.6" y="25.4" size="1.778" layer="95"/>
 </segment>
+<segment>
+<pinref part="J2" gate="G$1" pin="5"/>
+<wire x1="129.54" y1="73.66" x2="127" y2="73.66" width="0.1524" layer="91"/>
+<label x="121.92" y="73.66" size="1.778" layer="95"/>
+</segment>
 </net>
 <net name="LED1" class="0">
-<segment>
-<pinref part="J2" gate="G$1" pin="3"/>
-<wire x1="129.54" y1="78.74" x2="127" y2="78.74" width="0.1524" layer="91"/>
-<label x="121.92" y="78.74" size="1.778" layer="95"/>
-</segment>
 <segment>
 <pinref part="R1" gate="G$1" pin="1"/>
@@
 <label x="101.6" y="40.64" size="1.778" layer="95"/>
 </segment>
-</net>
-<net name="LOG" class="0">
 <segment>
 <pinref part="J2" gate="G$1" pin="4"/>
@@
 <label x="121.92" y="76.2" size="1.778" layer="95"/>
 </segment>
+</net>
+<net name="LOG" class="0">
 <segment>
 <pinref part="LOG" gate="G$1" pin="C@1"/>
@@
 <label x="10.16" y="27.94" size="1.778" layer="95"/>
 </segment>
+<segment>
+<pinref part="J2" gate="G$1" pin="3"/>
+<wire x1="129.54" y1="78.74" x2="127" y2="78.74" width="0.1524" layer="91"/>
+<label x="121.92" y="78.74" size="1.778" layer="95"/>
+</segment>
 </net>
 <net name="MARK" class="0">
-<segment>
-<pinref part="J2" gate="G$1" pin="5"/>
-<wire x1="129.54" y1="73.66" x2="127" y2="73.66" width="0.1524" layer="91"/>
-<label x="121.92" y="73.66" size="1.778" layer="95"/>
-</segment>
 <segment>
 <pinref part="MARK" gate="G$1" pin="C@2"/>
@@
 <label x="10.16" y="12.7" size="1.778" layer="95"/>
 </segment>
+<segment>
+<pinref part="J2" gate="G$1" pin="2"/>
+<wire x1="129.54" y1="81.28" x2="127" y2="81.28" width="0.1524" layer="91"/>
+<label x="119.38" y="81.28" size="1.778" layer="95"/>
+</segment>
 </net>
 <net name="RESET" class="0">
-<segment>
-<pinref part="J2" gate="G$1" pin="6"/>
-<wire x1="129.54" y1="71.12" x2="127" y2="71.12" width="0.1524" layer="91"/>
-<label x="121.92" y="71.12" size="1.778" layer="95"/>
-</segment>
 <segment>
 <pinref part="RESET" gate="G$1" pin="C@2"/>
@@
 <label x="10.16" y="-2.54" size="1.778" layer="95"/>
 </segment>
-</net>
+<segment>
+<pinref part="J2" gate="G$1" pin="1"/>
+<wire x1="129.54" y1="83.82" x2="127" y2="83.82" width="0.1524" layer="91"/>
+<label x="119.38" y="83.82" size="1.778" layer="95"/>
+</segment>
+</net>
