File: EAGLE/projects/CAN-D Rev2/CAN-D Rev2.brd (EAGLE design)
At the start: 55.3 x 80.3 mm, 34 parts, among them P1 TSM-106-SV, P2 TSM-106-SV, U1 TPS2115ADRBR, U2 MCP2562-E/SN, U3 FGPMMOPA6H, U4 STM32F302CCT6, X1 DX4R005HJ5R2000, X2 DM1AA-SF-PEJ(21), X3 1-1740195-2, Y1 ABLS-8.000MHZ-B2-T

Commit message: Clean up EAGLE files
Parts:
- removed VR: LD39200PU33R, LD39200PU33R:SON95P300X300X100-7N
- added C19, C20: 10u, rcl:C0603
- added VR1: 3.3V-REGULATOR, CAN-D:LD39200PU33R
- added VR2: 5V-REGULATOR, CAN-D:LD1086D2T50TR
- F1: value 0ZCJ0025FF2E -> FUSE; device 0ZCJ0025FF2E:RESC3216X125N -> CAN-D:0ZCJ0025FF2E
- P1, P2: value TSM-106-SV -> HEADER; device con-samtec:TSM-106-SV -> CAN-D:TSM-106-02-L-SV-P-TR
- U1: value TPS2115ADRBR -> POWER-MUX; device TPS2115ADRBR:SON65P300X300X100-9N -> CAN-D:TPS2115ADRBR
- U2: value MCP2562-E/SN -> CAN-TRANSCEIVER; device MCP2562-E_SN:SOIC127P600X175-8N -> CAN-D:MCP2562-E/SN
- U3: value FGPMMOPA6H -> GPS; device FGPMMOPA6H:FGPMMOPA6H -> CAN-D:FGPMMOPA6H
- U4: value STM32F302CCT6 -> MCU; device STM32F302CCT6:QFP50P900X900X160-48N -> CAN-D:STM32F302CCT6
- X1: value DX4R005HJ5R2000 -> MICRO-USB; device DX4R005HJ5R2000:JAE_DX4R005HJ5R2000 -> CAN-D:DX4R005HJ5R2000
- X2: value DM1AA-SF-PEJ(21) -> SD-READER; device DM1AA-SF-PEJ_21_:HRS_DM1AA-SF-PEJ(21) -> CAN-D:DM1AA-SF-PEJ(21)
- X3: value 1-1740195-2 -> DB9; device 1-1740195-2:1-1740195-2 -> CAN-D:1-1740195-2
- Y1: value ABLS-8.000MHZ-B2-T -> OSCILLATOR; device ABLS-8.000MHZ-B2-T:XTAL_ABLS-8.000MHZ-B2-T -> CAN-D:ABLS-8.000MHZ-B2-T
- moved X3 9.35 mm to (18.4, -7.72)
- moved P2 3.11 mm to (37.3, 18.3)
Connections:
- new net N$3: C1.1, C20.1, U1.8, VR2.TAB
- net DB9VCC: now also C19.1, VR2.3; no longer C1.1, U1.8
- net GND: now also C19.2, C20.2, VR1.3, VR1.7, VR2.1; no longer VR.3, VR.7
- net N$1: now also VR1.5, VR1.6; no longer VR.5, VR.6
- net VCC: now also VR1.1, VR1.2; no longer VR.1, VR.2
Routing:
- net N$3: track 0.00 -> 51.5 mm
- net DB9VCC: track 78.4 -> 36.4 mm
- net N$7: track 61.1 -> 69.5 mm, vias 0 -> 2
- net N$2: track 67.4 -> 75.6 mm, vias 0 -> 2
- net LED2: track 18.1 -> 11.2 mm
- net LOG: track 18.0 -> 11.2 mm
- net RESET: track 41.3 -> 45.8 mm
- net GND: track 18.6 -> 22.9 mm, vias 6 -> 16
- net VCC: track 159.1 -> 163.3 mm, vias 6 -> 4
- net SYS_JTMS-SWDIO: track 16.2 -> 20.0 mm
- net SYS_JTDO-TRACESWO: track 19.0 -> 22.8 mm
- net SYS_JTCK-SWCLK: track 23.4 -> 19.7 mm
- net SYS_NJTRST: track 20.5 -> 19.3 mm
- net LED1: track 14.2 -> 14.9 mm
- net LED3: track 16.0 -> 16.6 mm

Commit message: Upload Final Revisions to Board Design
Connections:
- net GND: now also X3.3
Routing:
- net DB9VCC: track 36.4 -> 28.2 mm
- net N$7: track 69.5 -> 74.6 mm
- net N$2: track 75.6 -> 78.3 mm
Changed lines of the file:
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@@
 <?xml version="1.0" encoding="utf-8"?>
 <!DOCTYPE eagle SYSTEM "eagle.dtd">
-<eagle version="9.3.1">
+<eagle version="9.3.2">
 <drawing>
 <settings>
-<setting alwaysvectorfont="no"/>
+<setting alwaysvectorfont="yes"/>
 <setting verticaltext="up"/>
 </settings>
@@
 </layers>
 <board>
-<fusionsync huburn="a.cGVyc29uYWw6dWUyYzU5ZGVl" projecturn="a.cGVyc29uYWw6dWUyYzU5ZGVlIzIwMTkwMzIyMTgzOTA3OTUx" f3durn="urn:adsk.wipprod:dm.lineage:dNOZHJjHQz-2HrBDH3L1DQ" pcbguid="1b160407-f627-4c7c-9021-4d10ae83106a" lastpulledtime="2019-03-23T12:45:51Z" lastsyncedchangeguid="344d305b-5af5-8e0d-6624-3849b992070b"/>
+<fusionsync huburn="a.cGVyc29uYWw6dWUyYzU5ZGVl" projecturn="a.cGVyc29uYWw6dWUyYzU5ZGVlIzIwMTkwMzIyMTgzOTA3OTUx" f3durn="urn:adsk.wipprod:dm.lineage:dNOZHJjHQz-2HrBDH3L1DQ" pcbguid="1b160407-f627-4c7c-9021-4d10ae83106a" lastpulledtime="2019-03-23T12:45:51Z" lastsyncedchangeguid="458a52d9-ed36-dab9-cc35-98f93087e69c"/>
 <plain>
 <text x="1.3462" y="37.4142" size="1.778" layer="21">CAN-D
@@
 <wire x1="43.047" y1="35.9664" x2="43.8912" y2="35.9664" width="0.2794" layer="16"/>
 <via x="43.8912" y="35.9664" extent="1-16" drill="0.35"/>
+<contactref element="X3" pad="3"/>
 </signal>
 <signal name="USBVCC">
@@
 <signal name="DB9VCC">
 <contactref element="X3" pad="9"/>
-<wire x1="14.33" y1="5.378" x2="17.0672" y2="2.6416" width="0.6096" layer="1"/>
 <contactref element="VR2" pad="3"/>
 <contactref element="C19" pad="1"/>
-<wire x1="17.0672" y1="2.6416" x2="26.6192" y2="2.6416" width="0.6096" layer="1"/>
 <via x="26.6192" y="2.6416" extent="1-16" drill="0.35"/>
 <wire x1="35.9664" y1="2.4384" x2="35.7632" y2="2.6416" width="0.6096" layer="16"/>
@@
 <wire x1="39.3568" y1="10.84458125" x2="39.3568" y2="6.9824" width="0.6096" layer="1"/>
 <wire x1="39.3568" y1="6.9824" x2="37.15" y2="4.775" width="0.6096" layer="1"/>
+<wire x1="22.55" y1="5.378" x2="25.2864" y2="2.6416" width="0.6096" layer="1"/>
+<wire x1="25.2864" y1="2.6416" x2="26.6192" y2="2.6416" width="0.6096" layer="1"/>
 </signal>
 <signal name="N$1">
@@
 <wire x1="52.0328" y1="46.4684" x2="48.997" y2="46.468" width="0.6096" layer="1"/>
 <via x="27.6352" y="7.9248" extent="1-16" drill="0.35"/>
-<wire x1="19.81" y1="5.378" x2="21.7032" y2="7.2712" width="0.6096" layer="1"/>
 <wire x1="25.97298125" y1="7.9248" x2="27.6352" y2="7.9248" width="0.6096" layer="1"/>
 <wire x1="25.31938125" y1="7.2712" x2="25.97298125" y2="7.9248" width="0.6096" layer="1"/>
-<wire x1="21.7032" y1="7.2712" x2="25.31938125" y2="7.2712" width="0.6096" layer="1"/>
 <via x="52.0328" y="46.4684" extent="1-16" drill="0.35"/>
+<wire x1="21.96978125" y1="7.2712" x2="25.31938125" y2="7.2712" width="0.6096" layer="1"/>
 <wire x1="52.0328" y1="46.4684" x2="52.0328" y2="45.14980625" width="0.6096" layer="16"/>
 <wire x1="52.0328" y1="45.14980625" x2="52.7812" y2="44.40140625" width="0.6096" layer="16"/>
@@
 <wire x1="51.136675" y1="11.7856" x2="35.56" y2="11.7856" width="0.6096" layer="16"/>
 <wire x1="52.7812" y1="44.40140625" x2="52.7812" y2="13.430125" width="0.6096" layer="16"/>
+<wire x1="18.9628" y1="7.2708" x2="17.07" y2="5.378" width="0.6096" layer="1"/>
+<wire x1="21.96978125" y1="7.2712" x2="21.96938125" y2="7.2708" width="0.6096" layer="1"/>
+<wire x1="21.96938125" y1="7.2708" x2="18.9628" y2="7.2708" width="0.6096" layer="1"/>
 </signal>
 <signal name="N$7">
@@
 <wire x1="51.7652" y1="44.164125" x2="51.160925" y2="44.7684" width="0.6096" layer="1"/>
 <wire x1="51.160925" y1="44.7684" x2="48.997" y2="44.768" width="0.6096" layer="1"/>
-<wire x1="22.36501875" y1="10.7388" x2="21.1804" y2="9.55418125" width="0.6096" layer="1"/>
-<wire x1="21.18" y1="8.778" x2="21.1804" y2="9.55418125" width="0.6096" layer="1"/>
-<wire x1="22.36501875" y1="10.7388" x2="32.6844" y2="10.7388" width="0.6096" layer="1"/>
 <wire x1="32.6844" y1="10.7388" x2="33.3248" y2="11.3792" width="0.6096" layer="1"/>
 <via x="33.3248" y="11.3792" extent="1-16" drill="0.35"/>
@@
 <via x="51.7652" y="44.164125" extent="1-16" drill="0.35"/>
 <wire x1="34.544" y1="12.5984" x2="50.8" y2="12.5984" width="0.6096" layer="16"/>
+<wire x1="15.7" y1="8.778" x2="17.6608" y2="10.7388" width="0.6096" layer="1"/>
+<wire x1="17.6608" y1="10.7388" x2="32.6844" y2="10.7388" width="0.6096" layer="1"/>
 </signal>
 <signal name="CAN_STBY">
