File: EAGLE/projects/CAN-D Rev2/CAN-D Rev2.sch (EAGLE design)
At the start: 34 parts, among them P1 TSM-106-SV, P2 TSM-106-SV, U1 TPS2115ADRBR, U2 MCP2562-E/SN, U3 FGPMMOPA6H, U4 STM32F302CCT6, X1 DX4R005HJ5R2000, X2 DM1AA-SF-PEJ(21), X3 1-1740195-2, Y1 ABLS-8.000MHZ-B2-T

Commit message: Clean up EAGLE files
Parts:
- removed VR: LD39200PU33R, LD39200PU33R:LD39200PU33R
- added C19, C20: 10u, rcl:C-EUC0603
- added VR1: 3.3V-REGULATOR, CAN-D:3.3V-REGULATOR
- added VR2: 5V-REGULATOR, CAN-D:5V-REGULATOR
- F1: value 0ZCJ0025FF2E -> FUSE; device 0ZCJ0025FF2E:0ZCJ0025FF2E -> CAN-D:FUSE
- P1, P2: value TSM-106-SV -> HEADER; device con-samtec:TSM-106-SV -> CAN-D:HEADER
- U1: value TPS2115ADRBR -> POWER-MUX; device TPS2115ADRBR:TPS2115ADRBR -> CAN-D:POWER-MUX
- U2: value MCP2562-E/SN -> CAN-TRANSCEIVER; device MCP2562-E_SN:MCP2562-E/SN -> CAN-D:CAN-TRANSCEIVER
- U3: value FGPMMOPA6H -> GPS; device FGPMMOPA6H:FGPMMOPA6H -> CAN-D:GPS
- U4: value STM32F302CCT6 -> MCU; device STM32F302CCT6:STM32F302CCT6 -> CAN-D:MCU
- X1: value DX4R005HJ5R2000 -> MICRO-USB; device DX4R005HJ5R2000:DX4R005HJ5R2000 -> CAN-D:MICRO-USB
- X2: value DM1AA-SF-PEJ(21) -> SD-READER; device DM1AA-SF-PEJ_21_:DM1AA-SF-PEJ(21) -> CAN-D:SD-READER
- X3: value 1-1740195-2 -> DB9; device 1-1740195-2:1-1740195-2 -> CAN-D:DB9
- Y1: value ABLS-8.000MHZ-B2-T -> OSCILLATOR; device ABLS-8.000MHZ-B2-T:ABLS-8.000MHZ-B2-T -> CAN-D:OSCILLATOR
Connections:
- new net N$3: C1.1, C20.1, U1.IN1, VR2.OUT
- net DB9VCC: now also C19.1, VR2.IN; no longer C1.1, U1.IN1
- net GND: now also C19.2, C20.2, VR1.EPAD, VR1.GND, VR2.GND; no longer VR.EPAD, VR.GND
- net N$1: now also VR1.EN, VR1.IN; no longer VR.EN, VR.IN
- net VCC: now also VR1.ADJ/SENSE, VR1.OUT; no longer VR.ADJ/SENSE, VR.OUT
Other:
- moved on the sheet: C1, C10, C3, C5, F1, R5, U1

Commit message: Upload Final Revisions to Board Design
Connections:
- net GND: now also X3.3
Changed lines of the file:
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@@
 <part name="GND12" library="supply1" library_urn="urn:adsk.eagle:library:371" deviceset="GND" device=""/>
 <part name="C20" library="rcl" library_urn="urn:adsk.eagle:library:334" deviceset="C-EU" device="C0603" package3d_urn="urn:adsk.eagle:package:23616/2" value="10u"/>
+<part name="GND28" library="supply1" library_urn="urn:adsk.eagle:library:371" deviceset="GND" device=""/>
 </parts>
 <sheets>
@@
 <attribute name="NAME" x="230.124" y="140.081" size="1.778" layer="95"/>
 <attribute name="VALUE" x="230.124" y="135.001" size="1.778" layer="96"/>
+</instance>
+<instance part="GND28" gate="1" x="25.4" y="142.24" smashed="yes" rot="MR0">
+<attribute name="VALUE" x="22.86" y="147.32" size="1.778" layer="96" rot="MR180"/>
 </instance>
 </instances>
@@
 <pinref part="C20" gate="G$1" pin="2"/>
 </segment>
+<segment>
+<pinref part="X3" gate="G$1" pin="3"/>
+<pinref part="GND28" gate="1" pin="GND"/>
+<wire x1="30.48" y1="144.78" x2="25.4" y2="144.78" width="0.1524" layer="91"/>
+</segment>
 </net>
